File: Target.kicad_sch (KiCad schematic)
At the start: 43 parts, among them J3 CONN_Header_2Pin_2.54mmPitch, J4 ARM_SWD_SERIAL_10, J5 CONN_USB4155_USB_C_Plug, Q1 2N7002, Q2 2N7002, Q3 2N7002, Q4 2N7002, U1 EMI2121MTTAG, U6 PAC1921-1, U7 AP22814AW5, U8 IC_FSUSB42MUX

Commit message: Changes and updates for revision 1 release
Parts:
- removed R25: 0, Redhill_lib:R_0402_1005Metric, symbol Redhill_Lib:R_CHIP_0402_0
- removed U6: PAC1921-1, Redhill_lib:VDFN-10-1EP_3x3mm_P0.5mm_EP1.7x2.4mm, symbol Redhill_Lib:IC_PAC1921-1
- added C38, C43: 1uF, Redhill_lib:C_0402_1005Metric, symbol Redhill_Lib:CAP_CER_0402_1uF_16V_10%_X5R
- added C39: 10uF, Redhill_lib:C_0603_1608Metric, symbol Redhill_Lib:CAP_CER_0603_10uF_25V_20%_X5R
- added R14, R15: 12k, Redhill_lib:R_0402_1005Metric, symbol Redhill_Lib:R_CHIP_0402_12k_1%
- added R25: 100, Redhill_lib:R_0402_1005Metric, symbol Redhill_Lib:R_CHIP_0402_100_1%_0.0625W
- added R43: 51, Redhill_lib:R_0402_1005Metric, symbol Redhill_Lib:R_CHIP_0402_51_5%_0.0625W
- added R44, R51: 56k, Redhill_lib:R_0402_1005Metric, symbol Redhill_Lib:R_CHIP_0402_56k_5%
- added R46: 10k, Redhill_lib:R_0402_1005Metric, symbol Redhill_Lib:R_CHIP_0402_10k_1%
- added U11: FUSB303BTMX, Redhill_lib:Texas_X2QFN-12_1.6x1.6mm_P0.4mm, symbol Redhill_Lib:FUSB303BTMX
- added U6: IC_INA225, Redhill_lib:VSSOP-8_3.0x3.0mm_P0.65mm, symbol Redhill_Lib:IC_INA225
- R30: LCSC C2889962 -> C7500253; Partnumber ERJ-3EKF1004V -> CSR1206FK20L0
- renumbered FB1 to FB2, U1 to U9
Connections:
- net +3.3V: now also C38.1, C39.1, C43.2, R46.1, U11.12 (VDD), U6.3 (V_{S}), U6.5 (GS0)
- net +5V: now also U6.1 (IN+)
- net +5V_TARGET: now also U6.8 (IN-)
- net +5V_TARGET_SW: now also R14.1
- net GND: now also C38.2, C39.2, C43.1, R15.2, R44.2, R51.2, U11.10 (GND), U11.11 (EN_N), U6.2 (GND), U6.6 (GS1), U6.7 (REF)
- net I2C_SCL: now also U11.8 (SCL)
- net I2C_SDA: now also U11.7 (SDA)
- net OUT: now also R25.2, U6.4 (OUT)
- net TRGT_SWDCLK: now also D5.4 (K3); no longer D5.7 (K6)
- net UART_TARGET_RX: now also R44.1
- net USBC_TRG_PWR: now also U11.4 (VBUS_DET)
- net TRGT_PD: now reaches J4.7 (Presence_Detect)
- net TRGT_PD: now also D5.7 (K6), R43.2
- net TARGET_PRESENT renamed TARGET_PWR_ON
- net USBC_CC renamed DFP_CC1
- net DFP_CC1: now also U11.1 (CC1)
- net USBC_VCONN renamed DFP_CC2
- net DFP_CC2: now also U11.2 (CC2)
- new net: R51.1, U11.5 (ADDR/ORIENT)
- new net PD_DFP_INT: R46.2, U11.6 (INT_N)
- new net PWR_MON_ADC_I: R25.1
- new net PWR_MON_ADC_V: R14.2, R15.1
- new net TARGET_PRESENCE: R43.1
- no-connect marks 10 -> 12
Other:
- note added: "Gain set to 50V/V With 0.02Ohm sense resistor this equates to an output of 1V/A"
- note added: "I2C Addr (7-bit): 0x21"
- company: (none) -> Redhill Embedded
- title: (none) -> Magnum
- moved on the sheet: C34, C35, C36, J3, Q1, Q2, Q3, Q4, R22, R23, R24, R26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
