File: input.kicad_sch (KiCad schematic)
At the start: 37 parts, among them J1 USB_C_Receptacle_USB2.0, U1 EMI2121MTTAG, U2 IC_USB2412-DZK, U3 3.3V, 300mA, Y1 24MHz

Commit message: Changes and updates for revision 1 release
Parts:
- removed R14 (x2): 10k, Redhill_lib:R_0402_1005Metric, symbol Redhill_Lib:R_CHIP_0402_10k_1%
- added C40: 1uF, Redhill_lib:C_0402_1005Metric, symbol Redhill_Lib:CAP_CER_0402_1uF_16V_10%_X5R
- added C41: 10uF, Redhill_lib:C_0603_1608Metric, symbol Redhill_Lib:CAP_CER_0603_10uF_25V_20%_X5R
- added H1, H2: MountingHole, MountingHole:MountingHole_2.5mm, symbol Mechanical:MountingHole
- added R45: 10k, Redhill_lib:R_0402_1005Metric, symbol Redhill_Lib:R_CHIP_0402_10k_1%
- added U10: FUSB302BMPX, Redhill_lib:WQFN-14-1EP_2.5x2.5mm_P0.5mm_EP1.45x1.45mm, symbol Redhill_Lib:IC_FUSB302BMPX
- J1: Alternate LCSC (none) -> C2982555; Alternate Partnumber (none) -> TYPEC-304-ACP16
- renumbered D6 to D7, FB3 to FB7, FB3 to FB8, R41 to R47, R41 to R48
Connections:
- net +3.3V: now also C40.1, C41.1, R45.1, U10.12 (VCONN), U10.13 (VCONN), U10.3 (VDD), U10.4 (VDD)
- net +5V: now also U10.2 (VBUS)
- net GND: now also C40.2, C41.2, U10.15 (GND), U10.8 (GND), U10.9 (GND)
- net PROBE_CC1: now also U10.10 (CC1), U10.11 (CC1)
- net PROBE_CC2: now also U10.1 (CC2), U10.14 (CC2)
- new net I2C_SCL: U10.6 (SCL)
- new net I2C_SDA: U10.7 (SDA)
- new net PD_UFP_INT: R45.2, U10.5 (INT_N)
Other:
- note added: "I2C addr (7-bit): 0x22"
- company: (none) -> Redhill Embedded
- title: (none) -> Magnum
