File: magnum.kicad_pcb (KiCad board)
At the start: 4 copper layers, 62 x 27 mm, 118 parts, among them J1 USB_C_Receptacle_USB2.0, J2 Conn_ARM_SWD_TagConnect_TC203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, J3 CONN_Header_2Pin_2.54mmPitch, J4 ARM_SWD_SERIAL_10, J5 CONN_USB4155_USB_C_Plug, Q1 2N7002, Q2 2N7002, Q3 2N7002, Q4 2N7002, U1 EMI2121MTTAG, U2 IC_USB2412-DZK, U3 3.3V, 300mA, U4 W25Q32JVZP, U5 RP2040, U6 PAC1921-1, U7 AP22814AW5, U8 IC_FSUSB42MUX, U9 EMI2121MTTAG, Y1 24MHz, Y2 Crystal_ECS-120-20-33_12MHz

Commit message: Changes and updates for revision 1 release
Parts:
- removed D1: LTST-C190GKT, Redhill_lib:LED_0603_1608Metric
- removed J2: Conn_ARM_SWD_TagConnect_TC2030-NL, Connector:Tag-Connect_TC2030-IDC-NL_2x03_P1.27mm_Vertical
- added C38: 1uF, Redhill_lib:C_0402_1005Metric, B.Cu at (129.2, 98.2)
- added C39: 10uF, Redhill_lib:C_0603_1608Metric, B.Cu at (130.4, 97.8)
- added C40: 1uF, Redhill_lib:C_0402_1005Metric, F.Cu at (91.9, 99.0)
- added C41: 10uF, Redhill_lib:C_0603_1608Metric, B.Cu at (93.2, 97.6)
- added C42: 1uF, Redhill_lib:C_0402_1005Metric, F.Cu at (95.8, 97.2)
- added C43: 1uF, Redhill_lib:C_0402_1005Metric, F.Cu at (135.6, 113.4)
- added D8: LED_DUAL_RED_GREEN_LTST-C235KGKRKT, Redhill_lib:LED_LiteOn_LTST-C155GEKT, F.Cu at (103.7, 110.7)
- added H1: MountingHole, MountingHole:MountingHole_2.5mm, F.Cu at (104.0, 97.0)
- added H2: MountingHole, MountingHole:MountingHole_2.5mm, F.Cu at (139.0, 113.0)
- added J6: ARM_SWD_SERIAL_10, Redhill_lib:PinHeader_2x05_P1.27mm_Vertical_SMD, F.Cu at (85.3, 92.8)
- added R43: 51, Redhill_lib:R_0402_1005Metric, F.Cu at (125.4, 94.6)
- added R44: 56k, Redhill_lib:R_0402_1005Metric, B.Cu at (117.0, 107.2)
- added R45: 10k, Redhill_lib:R_0402_1005Metric, F.Cu at (98.0, 105.5)
- added R46: 10k, Redhill_lib:R_0402_1005Metric, B.Cu at (123.0, 104.3)
- added R51: 56k, Redhill_lib:R_0402_1005Metric, B.Cu at (124.2, 104.3)
- added R52: 100, Redhill_lib:R_0402_1005Metric, F.Cu at (99.1, 110.5)
- added U10: FUSB302BMPX, Redhill_lib:WQFN-14-1EP_2.5x2.5mm_P0.5mm_EP1.45x1.45mm, F.Cu at (91.9, 96.1)
- added U11: FUSB303BTMX, Redhill_lib:Texas_X2QFN-12_1.6x1.6mm_P0.4mm, B.Cu at (128.4, 100.7)
- added U12: IC_MEM_AT24CSW010-STUM-T, Redhill_lib:SOT-23-5, F.Cu at (98.3, 97.1)
- C34, R40: moved to F.Cu
- C36, R10, R2, R29: moved to B.Cu
- R14, R15: value 10k -> 12k
- R25: value 0 -> 100
- U4: footprint Package_SON:WSON-8-1EP_6x5mm_P1.27mm_EP3.4x4.3mm -> Redhill_lib:USON-8_2x3mm
- U6: value PAC1921-1 -> IC_INA225; footprint Redhill_lib:VDFN-10-1EP_3x3mm_P0.5mm_EP1.7x2.4mm -> Redhill_lib:VSSOP-8_3.0x3.0mm_P0.65mm
- Y2: footprint Redhill_lib:Crystal_SMD_0603-4Pin_6.0x3.5mm -> Redhill_lib:Crystal_SMD_3225-4Pin_3.2x2.5mm
- moved R49 20.3 mm to (105.2, 107.6)
- moved R50 16.2 mm to (106.7, 107.6), turned to 90 degrees
- moved R14 13.1 mm to (128.7, 104.2), turned to 180 degrees
- moved R27 12.6 mm to (123.6, 108.0), turned to 0 degrees
- moved R25 12.3 mm to (111.3, 108.0), turned to -90 degrees
- moved R40 11.8 mm to (126.0, 106.7), turned to 90 degrees
- moved J3 10.3 mm to (137.9, 108.8), turned to 0 degrees
- moved R31 10.2 mm to (123.6, 106.9)
- moved R15 9.09 mm to (126.4, 104.2), turned to 180 degrees
- moved U7 8.50 mm to (128.4, 107.2), turned to -90 degrees
- moved R20 7.83 mm to (100.0, 92.4)
- moved C34 7.82 mm to (134.6, 113.4), turned to 90 degrees
- moved R18 7.64 mm to (100.0, 93.6)
- moved C36 5.79 mm to (134.3, 110.0), turned to 90 degrees
- moved U6 5.69 mm to (132.2, 111.9), turned to 90 degrees
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Connections:
- net /Input/PROBE_DEBUG_RX renamed /MCU/UART_DEBUG_RX
- net /Input/PROBE_DEBUG_TX renamed /MCU/UART_DEBUG_TX
- net /MCU/TARGET_PRESENT renamed /MCU/TARGET_PWR_ON
- D5 pad 4: unconnected-(D5-K3-Pad4) -> /Target/TRGT_SWDCLK
- D5 pad 7: /Target/TRGT_SWDCLK -> /Target/TRGT_PD
- FB5 pad 1: /MCU/USBC_CC -> /Target/DFP_CC1
- FB6 pad 1: /MCU/USBC_VCONN -> /Target/DFP_CC2
- J4 pad 7: unconnected-(J4-KEY-Pad7) -> /Target/TRGT_PD
- R14 pad 1: +3.3V -> /Target/+5V_TARGET_SW
- R14 pad 2: /MCU/I2C_SDA -> /MCU/PWR_MON_ADC_V
- R15 pad 1: +3.3V -> /MCU/PWR_MON_ADC_V
- R15 pad 2: /MCU/I2C_SCL -> GND
- R18 pad 2: GND -> +3.3V
- R20 pad 2: GND -> +3.3V
- R25 pad 1: /Target/ADDR -> /MCU/PWR_MON_ADC_I
- R25 pad 2: GND -> /Target/OUT
- R49 pad 1: /Input/PROBE_CC1 -> +3.3V
- R49 pad 2: GND -> /MCU/I2C_SCL
- R50 pad 2: /Input/PROBE_CC2 -> /MCU/I2C_SDA
- U5 pad 13: /MCU/USBC_CC -> /Input/PD_UFP_INT
- U5 pad 14: /MCU/USBC_VCONN -> /MCU/PD_DFP_INT
- U5 pad 28: /MCU/STATUS_LED -> /MCU/DAP_STATE
- U5 pad 29: /MCU/DAP_STATE -> /MCU/TX_IND
- U5 pad 30: /MCU/TX_IND -> /MCU/RX_IND
- U5 pad 31: /MCU/RX_IND -> /MCU/STATUS_GREEN
- U5 pad 32: unconnected-(U5-GPIO21-Pad32) -> /MCU/STATUS_RED
- U5 pad 34: unconnected-(U5-GPIO22-Pad34) -> /MCU/PCA_ID_0
- U5 pad 35: unconnected-(U5-GPIO23-Pad35) -> /MCU/PCA_ID_1
- U5 pad 39: unconnected-(U5-GPIO27_ADC1-Pad39) -> /MCU/PWR_MON_ADC_V
- U5 pad 40: /MCU/PCA_ID_0 -> /MCU/PWR_MON_ADC_I
- U5 pad 41: /MCU/PCA_ID_1 -> unconnected-(U5-GPIO29_ADC3-Pad41)
- U5 pad 6: /MCU/PWR_MON_CTRL -> /MCU/TARGET_PRESENCE
- U6 pad 1: +3.3V -> +5V
- U6 pad 2: +5V -> GND
- U6 pad 3: /Target/+5V_TARGET -> +3.3V
- U6 pad 5: GND -> +3.3V
- U6 pad 6: /Target/ADDR -> GND
- U6 pad 7: unconnected-(U6-RESERVED-Pad7) -> GND
- U6 pad 8: /MCU/PWR_MON_CTRL -> /Target/+5V_TARGET
Routing:
- net /MCU/I2C_SCL: track 13.9 -> 64.2 mm, vias 2 -> 4
- net /Input/PD_UFP_INT: track 0.00 -> 48.0 mm, vias 0 -> 4
- net /MCU/I2C_SDA: track 13.9 -> 60.5 mm, vias 2 -> 4
- net /MCU/PWR_MON_ADC_V: track 0.00 -> 30.6 mm, vias 0 -> 2
- net /Target/OUT: track 1.30 -> 27.2 mm, vias 0 -> 1
- net /MCU/STATUS_RED: track 0.00 -> 24.1 mm, vias 0 -> 2
- net /MCU/STATUS_LED: track 23.6 -> 0.00 mm, vias 2 -> 0
- net /MCU/STATUS_GREEN: track 0.00 -> 20.3 mm, vias 0 -> 2
- net /MCU/TARGET_PRESENCE: track 0.00 -> 19.8 mm, vias 0 -> 2
- net /MCU/USBC_VCONN: track 17.7 -> 0.00 mm, vias 1 -> 0
- net GND: track 72.6 -> 89.9 mm, vias 83 -> 87
- net /MCU/TARGET_PWR_FAULT: track 29.5 -> 13.5 mm
- net /MCU/UART_DEBUG_TX: track 16.0 -> 31.5 mm
- net +5V: track 8.30 -> 23.6 mm
- net /MCU/USBC_CC: track 15.3 -> 0.00 mm, vias 1 -> 0
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- added copper zone on F.Cu, net GND
